File: Capacitive_Touch_Breakout_Board_AT42QT1245-AU.kicad_sch (KiCad schematic)
At the start: 41 parts, among them J101 Conn_01x10, SW101 Slider_7pos, SW102 Touchbutton, SW103 Slider_7pos, SW104 Touchbutton, SW105 Wheel_3pos, SW106 Touchbutton, SW107 Wheel_Interleaved_8pos, U101 AT42QT1245-AU, U102 UTC78L05_SOT89

Commit message: Annotations, ran ERC, fixed net Ry0 connected to Cs1 bug
Parts:
- added TP101, TP102, TP103, TP104, TP105, TP106, TP107, TP108, TP109, TP110: TestPoint, symbol Connector:TestPoint
Connections:
- net +5V: now also TP109.1
- net Cs0: now also TP107.1
- net GND: now also U101.3 (VSS), U101.5 (VSS), TP108.1, TP110.1
- net MISO: now also TP102.1
- net MOSI: now also TP103.1
- net Rx0: now also TP106.1
- net SCK: now also TP101.1
- net ~{DRDY}: now also TP105.1
- net ~{SS}: now also TP104.1
Other:
- note added: "2. Place TP? close to TP?"
- note added: "Note 2"
- note removed: "NEED TO ADD PWR TEST POINTS OUTPUT PIN FOR +5V"
- note removed: "NEED TO CONNECT PINS 3 & 5 TO GROUND"
- moved on the sheet: C102, R111, R112, SW101, SW102
